Commit message: URDF chanded

File: nda_robot_pkgs/nda_robot_description/urdf/past_robot.urdf (robot description, URDF)
Before this commit: robot nda_robot, 10 links, 9 joints
Links:
- removed link housing_link
- link base_link: mass None -> 20.0; geometry collision box size=1.0 0.4 1.0; visual box size=1.0 0.4 1.0
- link center_wheel_link: geometry collision cylinder length=0.05 radius=0.10; visual cylinder length=0.05 radius=0.10
Joints:
- removed joint base_link_to_housing_link
- joint base_link_to_base_footprint: origin xyz=0 0 0.15 -> xyz=0 0 0.65
- joint base_link_to_center_wheel_link: origin xyz=0.5 0 -0.075 rpy=-1.57 0 0 -> xyz=0.25 0 -0.55 rpy=-1.57 0 0
- joint base_link_to_imu_link: origin xyz=0 0 0.1 -> xyz=0 0 -0.1
- joint base_link_to_left_lrf_link: origin xyz=0 0.2305 0.2141 rpy=0 0 1.57 -> xyz=-0.25 0.2305 -0.3641 rpy=0 0 1.57
- joint base_link_to_left_wheel_link: origin xyz=0 0.24 0 rpy=1.57 0 0 -> xyz=-0.25 0.24 -0.5 rpy=-1.57 0 0
- joint base_link_to_lrf_link: origin xyz=0 0 0.2141 -> xyz=-0.25 0 -0.35
- joint base_link_to_right_lrf_link: origin xyz=0 -0.2305 0.2141 rpy=0 0 -1.57 -> xyz=-0.25 -0.2305 -0.3641 rpy=0 0 -1.57
- joint base_link_to_right_wheel_link: origin xyz=0 -0.24 0 rpy=1.57 0 0 -> xyz=-0.25 -0.24 -0.5 rpy=1.57 0 0
