Commit message: sensor dist chande

File: nda_robot_pkgs/nda_robot_description/urdf/robot.urdf (robot description, URDF)
Before this commit: robot nda_robot, 9 links, 8 joints
Joints:
- joint base_link_to_left_lrf_link: origin xyz=-0.25 0.3 -0.35 rpy=0 0 1.57 -> xyz=-0.25 0.2305 -0.35 rpy=0 0 1.57
- joint base_link_to_left_wheel_link: origin xyz=-0.25 0.3 -0.5 rpy=-1.57 0 0 -> xyz=-0.25 0.24 -0.5 rpy=-1.57 0 0
- joint base_link_to_right_lrf_link: origin xyz=-0.25 -0.3 -0.35 rpy=0 0 -1.57 -> xyz=-0.25 -0.2305 -0.35 rpy=0 0 -1.57
- joint base_link_to_right_wheel_link: origin xyz=-0.25 -0.3 -0.5 rpy=1.57 0 0 -> xyz=-0.25 -0.24 -0.5 rpy=1.57 0 0

Commit message: urdf修正

File: nda_robot_pkgs/nda_robot_description/urdf/robot.urdf (robot description, URDF)
Before this commit: robot nda_robot, 9 links, 8 joints
Joints:
- joint base_link_to_left_lrf_link: origin xyz=-0.25 0.2305 -0.35 rpy=0 0 1.57 -> xyz=-0.25 0.2305 -0.3641 rpy=0 0 1.57
- joint base_link_to_right_lrf_link: origin xyz=-0.25 -0.2305 -0.35 rpy=0 0 -1.57 -> xyz=-0.25 -0.2305 -0.3641 rpy=0 0 -1.57

Commit message: urdf modified

File: nda_robot_pkgs/nda_robot_description/urdf/robot.urdf (robot description, URDF)
Before this commit: robot nda_robot, 10 links, 9 joints
Links:
- link housing_link: geometry collision box size=0.9 0.4 1.0; visual box size=0.9 0.4 1.0

Commit message: add 3d_sensor_link

File: nda_robot_pkgs/nda_robot_description/urdf/robot.urdf (robot description, URDF)
Before this commit: robot nda_robot, 10 links, 9 joints
Links:
- added link threed_sensor_link
Joints:
- added joint base_link_to_threed_sensor_link: type fixed, parent base_link, child threed_sensor_link, origin xyz=0.7 0 0.22 

Commit message: urdf modified

File: nda_robot_pkgs/nda_robot_description/urdf/robot.urdf (robot description, URDF)
Before this commit: robot nda_robot, 11 links, 10 joints
Links:
- link housing_link: geometry collision box size=1.0 0.4 1.0; visual box size=1.0 0.4 1.0
Joints:
- joint base_link_to_threed_sensor_link: origin xyz=0.7 0 0.22  -> xyz=0.75 0 0.22 

Commit message: frame modified

File: nda_robot_pkgs/nda_robot_description/urdf/robot.urdf (robot description, URDF)
Before this commit: robot nda_robot, 11 links, 10 joints
Links:
- added link frame_link, mass 2.0; collision box size=0.88 0.4 0.775; visual box size=0.88 0.4 0.775
- link housing_link: mass 20.0 -> 18.0; geometry collision box size=1.075 0.4 0.265; visual box size=1.075 0.4 0.265
Joints:
- added joint base_link_to_frame_link: type fixed, parent base_link, child frame_link, origin xyz=0.15 0 0.652
- joint base_link_to_base_footprint: origin xyz=0 0 0.15 -> xyz=0 0 0.11
- joint base_link_to_housing_link: origin xyz=0.25 0 0.5 -> xyz=0.25 0 0.1325
- joint base_link_to_left_lrf_link: origin xyz=0 0.2305 0.2141 rpy=0 0 1.57 -> xyz=0 0.2305 0.137 rpy=0 0 1.57
- joint base_link_to_lrf_link: origin xyz=0 0 0.2141 -> xyz=0 0 0.137
- joint base_link_to_right_lrf_link: origin xyz=0 -0.2305 0.2141 rpy=0 0 -1.57 -> xyz=0 -0.2305 0.137 rpy=0 0 -1.57
- joint base_link_to_threed_sensor_link: origin xyz=0.75 0 0.22  -> xyz=0.60 0 0.265 
